File: sml_lesekopf.kicad_pcb (KiCad board)
At the start: 2 copper layers, 27 x 27 mm, 27 parts, among them Q1 BC807, Q2 SFH309, Q3 BC817, U1 74LVC1G17, U2 74LVC1G17, U3 MAX485E, U4 ADM3490ExR

Commit message: update pcb
Parts:
- added JP3: SolderJumper_3_Bridged12, Jumper:SolderJumper-3_P1.3mm_Bridged12_Pad1.0x1.5mm, B.Cu at (58.0, 54.4)
- moved Q3 0.85 mm to (64.8, 63.6)
- renumbered Vcc to J1, GND to J2, RX to J3, TX to J4, B to J5, A to J6, Z to J7, Y to J8
Connections:
- JP2 pad 1: VCC -> Net-(JP2-Pad1)
- U3 pad 3: VCC -> Net-(JP2-Pad1)
Routing:
- net Net-(JP2-Pad1): track 0.00 -> 6.86 mm, vias 0 -> 1
- net VCC: track 66.2 -> 69.0 mm, vias 2 -> 4
- net Net-(Q3-Pad3): track 8.00 -> 8.85 mm
- net Net-(Q2-Pad2): track 7.77 -> 8.62 mm
- net GND: track 68.9 -> 68.5 mm, vias 0 -> 1
Other:
- board text added: "A"
- board text added: "B"
- board text added: "RS485 RE/DE"
- board text added: "RX"
- board text added: "TX"
- board text added: "VCC"
- board text added: "X"
- board text added: "Y"
